Commit message: fixed transform tree

File: src/chassis/description/chassis_core.xacro (robot description, xacro)
@@ -18,11 +18,20 @@
     </material>
     <!-- BASE LINK -->
-    <link name="base_link"></link>
+    <link name="base_footprint"/>
     <joint name="base_footprint_joint" type="fixed">
-        <parent link="base_link"/>
-        <child link="base_footprint"/>
+        <parent link="base_footprint"/>
+        <child link="base_link"/>
         <origin xyz="0 0 0" rpy="0 0 0"/>
     </joint>
-    <link name="base_footprint"></link>
+    <link name="base_link">
+        <inertial>
+            <origin xyz="0 0 0" rpy="0 0 0"/>
+            <mass value="10.0"/>
+            <inertia
+            ixx="0.05" ixy="0.0" ixz="0.0"
+            iyy="0.05" iyz="0.0"
+            izz="0.05"/>
+        </inertial>
+    </link>
     <!-- CHASSIS LINK -->
     <joint name="chassis_joint" type="fixed">
@@ -53,9 +62,10 @@
         <parent link="base_link"/>
         <child link="left_wheel_link"/>
-        <origin xyz="0 -0.09144 -0.0127" rpy="-1.5707963267948966 0 0"/> <!-- Rotate wheel -->
-        <axis xyz="0 0 -1"/>
+        <origin xyz="0 -0.09144 -0.0127" rpy="0 0 0"/> <!-- Rotate wheel -->
+        <axis xyz="0 1 0"/>
     </joint>
     <link name="left_wheel_link">
         <visual>
+            <origin rpy="1.57079632679 0 0"/>
             <geometry>
                 <cylinder radius="0.0325" length="0.027"/>
@@ -76,9 +86,10 @@
         <parent link="base_link"/>
         <child link="right_wheel_link"/>
-        <origin xyz="0 0.09144 -0.0127" rpy="1.5707963267948966 0 0"/> <!-- Rotate wheel -->
-        <axis xyz="0 0 1"/>
+        <origin xyz="0 0.09144 -0.0127" rpy="0 0 0"/> <!-- Rotate wheel -->
+        <axis xyz="0 1 0"/>
     </joint>
     <link name="right_wheel_link">
         <visual>
+            <origin rpy="1.57079632679 0 0"/>
             <geometry>
                 <cylinder radius="0.0325" length="0.027"/>
@@ -118,4 +129,23 @@
         </xacro:inertial_sphere>
     </link>
+    <!-- GAZEBO FRICTION -->
+    <gazebo reference="left_wheel_link">
+        <mu1>1.0</mu1>      <!-- longitudinal friction -->
+        <mu2>1.0</mu2>      <!-- lateral friction -->
+        <kp>1000000.0</kp>  <!-- contact stiffness -->
+        <kd>1.0</kd>        <!-- damping -->
+    </gazebo>
+    <gazebo reference="right_wheel_link">
+        <mu1>1.0</mu1>
+        <mu2>1.0</mu2>
+        <kp>1000000.0</kp>
+        <kd>1.0</kd>
+    </gazebo>
+    <gazebo reference="caster_wheel_link">
+        <mu1>0.001</mu1>
+        <mu2>0.001</mu2>
+        <kp>1000000.0</kp>
+        <kd>1.0</kd>
+    </gazebo>
     <!-- LIDAR LINK -->
     <joint name="lidar_joint" type="fixed">
@@ -141,6 +171,6 @@
         <joint name="left_wheel_joint">
             <command_interface name="velocity">
-                <param name="min">-10</param>
-                <param name="max">10</param>
+                <param name="min">-1</param>
+                <param name="max">1</param>
             </command_interface>
             <state_interface name="velocity"/>
@@ -149,6 +179,6 @@
         <joint name="right_wheel_joint">
             <command_interface name="velocity">
-                <param name="min">-10</param>
-                <param name="max">10</param>
+                <param name="min">-1</param>
+                <param name="max">1</param>
             </command_interface>
             <state_interface name="velocity"/>
@@ -161,6 +191,3 @@
         </plugin>
     </gazebo>
-    <!-- <gazebo>
-        <plugin name="gazebo_ros2_control" filename="libgazebo_ros2_control.so"/>
-    </gazebo> -->
 </robot>

Commit message: updated urdf code

File: src/chassis/description/chassis_core.xacro (robot description, xacro)
@@ -2,4 +2,5 @@
 <robot xmlns:xacro="http://www.ros.org/wiki/xacro">
     <xacro:include filename="inertial_macros.xacro"/>
+    <!-- VISUAL COLORS -->
     <material name="white">
         <color rgba="1 1 1 1"/>
@@ -18,49 +19,82 @@
     </material>
     <!-- BASE LINK -->
-    <link name="base_footprint"/>
-    <joint name="base_footprint_joint" type="fixed">
-        <parent link="base_footprint"/>
-        <child link="base_link"/>
-        <origin xyz="0 0 0" rpy="0 0 0"/>
-    </joint>
-    <link name="base_link">
-        <inertial>
-            <origin xyz="0 0 0" rpy="0 0 0"/>
-            <mass value="10.0"/>
-            <inertia
-            ixx="0.05" ixy="0.0" ixz="0.0"
-            iyy="0.05" iyz="0.0"
-            izz="0.05"/>
-        </inertial>
-    </link>
+    <link name="base_link"></link>
     <!-- CHASSIS LINK -->
     <joint name="chassis_joint" type="fixed">
         <parent link="base_link"/>
         <child link="chassis_link"/>
-        <origin xyz="0.0508 0 0" rpy="0 0 0"/> <!-- Offset the chassis slightly back by 5.08cm-->
+        <origin xyz="0.196 0 0.075" rpy="0 0 0"/> <!-- Offset the chassis slightly up by 7.5cm-->
     </joint>
     <link name="chassis_link">
         <visual>
-            <origin xyz="-0.13462 0 0.06096" rpy="0 0 0"/>
-            <geometry>
-                <box size="0.26924 0.1524 0.12192"/>
+            <origin xyz="0 0 0" rpy="0 0 0"/>
+            <geometry>
+                <box size="0.392 0.29 0.06"/>
             </geometry>
             <material name="white"/>
         </visual>
         <collision>
-            <origin xyz="-0.13462 0 0.06096" rpy="0 0 0"/>
-            <geometry>
-                <box size="0.26924 0.1524 0.12192"/>
-            </geometry>
-        </collision>
-        <xacro:inertial_box mass="0.5" x="0.26924" y="0.1524" z="0.12192">
-            <origin xyz="-0.13462 0 0.06096" rpy="0 0 0"/>
+            <origin xyz="0 0 0" rpy="0 0 0"/>
+            <geometry>
+                <box size="0.392 0.29 0.06"/>
+            </geometry>
+            <material name="white"/>
+        </collision>
+        <xacro:inertial_box mass="0.5" x="0.392" y="0.29" z="0.06">
+            <origin xyz="0 0 0" rpy="0 0 0"/>
         </xacro:inertial_box>
     </link>
-    <!-- LEFT WHEEL LINK -->
+    <!-- POLE LINKS -->
+    <joint name="left_pole_joint" type="fixed">
+        <parent link="base_link"/>
+        <child link="left_pole_link"/>
+        <origin xyz="0 0.105 0.04" rpy="0 0 0"/>
+    </joint>
+    <link name="left_pole_link">
+        <visual>
+            <origin xyz="0 0 0.335" rpy="0 0 0"/>
+            <geometry>
+                <cylinder length="0.67" radius="0.00795"/>
+            </geometry>
+            <material name="black"/>
+        </visual>
+        <collision>
+            <origin xyz="0 0 0.335" rpy="0 0 0"/>
+            <geometry>
+                <cylinder length="0.67" radius="0.00795"/>
+            </geometry>
+        </collision>
+        <xacro:inertial_cylinder mass="0.02" length="0.67" radius="0.00795">
+            <origin xyz="0 0 0.335" rpy="0 0 0"/>
+        </xacro:inertial_cylinder>
+    </link>
+    <joint name="right_pole_joint" type="fixed">
+        <parent link="base_link"/>
+        <child link="right_pole_link"/>
+        <origin xyz="0 -0.105 0.04" rpy="0 0 0"/>
+    </joint>
+    <link name="right_pole_link">
+        <visual>
+            <origin xyz="0 0 0.335" rpy="0 0 0"/>
+            <geometry>
+                <cylinder length="0.67" radius="0.00795"/>
+            </geometry>
+            <material name="black"/>
+        </visual>
+        <collision>
+            <origin xyz="0 0 0.335" rpy="0 0 0"/>
+            <geometry>
+                <cylinder length="0.67" radius="0.00795"/>
+            </geometry>
+        </collision>
+        <xacro:inertial_cylinder mass="0.02" length="0.67" radius="0.00795">
+            <origin xyz="0 0 0.335" rpy="0 0 0"/>
+        </xacro:inertial_cylinder>
+    </link>
+    <!-- MOTOR WHEEL LINKS -->
     <joint name="left_wheel_joint" type="continuous">
         <parent link="base_link"/>
         <child link="left_wheel_link"/>
-        <origin xyz="0 -0.09144 -0.0127" rpy="0 0 0"/> <!-- Rotate wheel -->
+        <origin xyz="0.326 0.1685 0.034" rpy="0 0 0"/> <!-- Rotate wheel -->
         <axis xyz="0 1 0"/>
     </joint>
@@ -69,22 +103,22 @@
             <origin rpy="1.57079632679 0 0"/>
             <geometry>
-                <cylinder radius="0.0325" length="0.027"/>
+                <cylinder radius="0.034" length="0.026"/>
             </geometry>
             <material name="blue"/>
         </visual>
         <collision>
-            <geometry>
-                <cylinder radius="0.0325" length="0.027"/>
-            </geometry>
-        </collision>
-        <xacro:inertial_cylinder mass="0.1" length="0.027" radius="0.035">
-            <origin xyz="0 0 0" rpy="0 0 0"/>
-        </xacro:inertial_cylinder>
-    </link>
-    <!-- RIGHT WHEEL LINK -->
+            <origin rpy="1.57079632679 0 0"/>
+            <geometry>
+                <cylinder radius="0.034" length="0.026"/>
+            </geometry>
+        </collision>
+        <xacro:inertial_cylinder mass="0.02" radius="0.034" length="0.026">
+            <origin xyz="0 0 0" rpy="0 0 0"/>
+        </xacro:inertial_cylinder>
+    </link>
     <joint name="right_wheel_joint" type="continuous">
         <parent link="base_link"/>
         <child link="right_wheel_link"/>
-        <origin xyz="0 0.09144 -0.0127" rpy="0 0 0"/> <!-- Rotate wheel -->
+        <origin xyz="0.326 -0.1685 0.034" rpy="0 0 0"/> <!-- Rotate wheel -->
         <axis xyz="0 1 0"/>
     </joint>
@@ -93,37 +127,58 @@
             <origin rpy="1.57079632679 0 0"/>
             <geometry>
-                <cylinder radius="0.0325" length="0.027"/>
+                <cylinder radius="0.034" length="0.026"/>
             </geometry>
             <material name="blue"/>
         </visual>
         <collision>
-            <geometry>
-                <cylinder radius="0.0325" length="0.027"/>
-            </geometry>
-        </collision>
-        <xacro:inertial_cylinder mass="0.1" length="0.027" radius="0.035">
-            <origin xyz="0 0 0" rpy="0 0 0"/>
-        </xacro:inertial_cylinder>
-    </link>
-    <!-- CASTER WHEEL LINK -->
-    <joint name="caster_wheel_joint" type="fixed">
-        <parent link="base_link"/>
-        <child link="caster_wheel_link"/>
-        <origin xyz="-0.15 0 0" rpy="0 0 0"/>
-    </joint>
-    <link name="caster_wheel_link">
-        <visual>
-            <geometry>
-                <sphere radius="0.04572"/>
-            </geometry>
-            <material name="black"/>
-        </visual>
-        <collision>
-            <geometry>
-                <sphere radius="0.04572"/>
-            </geometry>
-            <material name="black"/>
-        </collision>
-        <xacro:inertial_sphere mass="0.1" radius="0.04572">
+            <origin rpy="1.57079632679 0 0"/>
+            <geometry>
+                <cylinder radius="0.034" length="0.026"/>
+            </geometry>
+        </collision>
+        <xacro:inertial_cylinder mass="0.02" radius="0.034" length="0.026">
+            <origin xyz="0 0 0" rpy="0 0 0"/>
+        </xacro:inertial_cylinder>
+    </link>
+    <!-- CASTER WHEELS LINK -->
+    <joint name="caster_left_wheel_joint" type="fixed">
+        <parent link="base_link"/>
+        <child link="caster_left_wheel_link"/>
+        <origin xyz="0 0.105 0.02" rpy="0 0 0"/>
+    </joint>
+    <link name="caster_left_wheel_link">
+        <visual>
+            <geometry>
+                <sphere radius="0.02"/>
+            </geometry>
+            <material name="black"/>
+        </visual>
+        <collision>
+            <geometry>
+                <sphere radius="0.02"/>
+            </geometry>
+        </collision>
+        <xacro:inertial_sphere mass="0.1" radius="0.02">
+            <origin xyz="0 0 0" rpy="0 0 0"/>
+        </xacro:inertial_sphere>
+    </link>
+    <joint name="caster_right_wheel_joint" type="fixed">
+        <parent link="base_link"/>
+        <child link="caster_right_wheel_link"/>
+        <origin xyz="0 -0.105 0.02" rpy="0 0 0"/>
+    </joint>
+    <link name="caster_right_wheel_link">
+        <visual>
+            <geometry>
+                <sphere radius="0.02"/>
+            </geometry>
+            <material name="black"/>
+        </visual>
+        <collision>
+            <geometry>
+                <sphere radius="0.02"/>
+            </geometry>
+        </collision>
+        <xacro:inertial_sphere mass="0.1" radius="0.02">
             <origin xyz="0 0 0" rpy="0 0 0"/>
         </xacro:inertial_sphere>
@@ -142,5 +197,5 @@
         <kd>1.0</kd>
     </gazebo>
-    <gazebo reference="caster_wheel_link">
+    <gazebo reference="caster_left_wheel_link">
         <mu1>0.001</mu1>
         <mu2>0.001</mu2>
@@ -148,48 +203,20 @@
         <kd>1.0</kd>
     </gazebo>
-    <!-- LIDAR LINK -->
-    <joint name="lidar_joint" type="fixed">
-        <parent link="base_link"/>
-        <child link="lidar_link"/>
-        <origin xyz="-0.06 0 0.13442" rpy="0 0 0"/>
-    </joint>
-    <link name="lidar_link">
-        <visual>
-            <geometry>
-                <cylinder radius="0.035" length="0.025"/>
-            </geometry>
-            <material name="red"/>
-        </visual>
-        <xacro:inertial_cylinder mass="0.140" length="0.025" radius="0.035">
-            <origin xyz="0 0 0" rpy="0 0 0"/>
-        </xacro:inertial_cylinder>
-    </link>
-    <plugin
-      filename="gz-sim-sensors-system"
-      name="gz::sim::systems::Sensors">
+    <gazebo reference="caster_right_wheel_link">
+        <mu1>0.001</mu1>
+        <mu2>0.001</mu2>
+        <kp>1000000.0</kp>
+        <kd>1.0</kd>
+    </gazebo>
+    <!-- GAZEBO PLUGINS -->
+    <plugin filename="gz-sim-sensors-system" name="gz::sim::systems::Sensors">
       <render_engine>ogre2</render_engine>
     </plugin>
-    <gazebo reference="lidar_link">
-        <sensor name="lidar_sensor" type="gpu_lidar">
-            <pose>0 0 0 0 0 0</pose>
-            <always_on>true</always_on>
-            <update_rate>10</update_rate>
-            <visualize>true</visualize>
-            <ray>
-                <scan>
-                    <horizontal>
-                    <samples>360</samples>
-                    <resolution>1</resolution>
-                    <min_angle>-3.14159</min_angle>
-                    <max_angle>3.14159</max_angle>
-                    </horizontal>
-                </scan>
-                <range>
-                    <min>0.3</min>
-                    <max>12.0</max>
-                </range>
-            </ray>
-        </sensor>
-    </gazebo>
+    <gazebo>
+        <plugin filename="gz_ros2_control-system" name="gz_ros2_control::GazeboSimROS2ControlPlugin">
+            <parameters>$(find chassis)/config/my_controllers.yaml</parameters>
+        </plugin>
+    </gazebo>
+    <!-- ROS CONTROL -->
     <ros2_control name="GazeboSimSystem" type="system">
         <hardware>
@@ -213,8 +240,3 @@
         </joint>
     </ros2_control>
-    <gazebo>
-        <plugin filename="gz_ros2_control-system" name="gz_ros2_control::GazeboSimROS2ControlPlugin">
-            <parameters>$(find chassis)/config/my_controllers.yaml</parameters>
-        </plugin>
-    </gazebo>
 </robot>

Commit message: added lidar link

File: src/chassis/description/chassis_core.xacro (robot description, xacro)
@@ -183,4 +183,21 @@
             <origin xyz="0 0 0" rpy="0 0 0"/>
         </xacro:inertial_sphere>
+    </link>
+    <!-- LIDAR LINK -->
+    <joint name="lidar_joint" type="fixed">
+        <parent link="base_link"/>
+        <child link="lidar_link"/>
+        <origin xyz="0.196 0 0.135" rpy="0 0 0"/>
+    </joint>
+    <link name="lidar_link">
+        <visual>
+            <geometry>
+                <cylinder radius="0.035" length="0.025"/>
+            </geometry>
+            <material name="red"/>
+        </visual>
+        <xacro:inertial_cylinder mass="0.140" length="0.025" radius="0.035">
+            <origin xyz="0 0 0" rpy="0 0 0"/>
+        </xacro:inertial_cylinder>
     </link>
     <!-- GAZEBO FRICTION -->
@@ -217,4 +234,27 @@
             <parameters>$(find chassis)/config/my_controllers.yaml</parameters>
         </plugin>
+    </gazebo>
+    <!-- GAZEBO LIDAR REFERENCE -->
+    <gazebo reference="lidar_link">
+        <sensor name="lidar_sensor" type="gpu_lidar">
+            <pose>0 0 0 0 0 0</pose>
+            <always_on>true</always_on>
+            <update_rate>10</update_rate>
+            <visualize>true</visualize>
+            <ray>
+                <scan>
+                    <horizontal>
+                    <samples>360</samples>
+                    <resolution>1</resolution>
+                    <min_angle>-3.14159</min_angle>
+                    <max_angle>3.14159</max_angle>
+                    </horizontal>
+                </scan>
+                <range>
+                    <min>0.3</min>
+                    <max>12.0</max>
+                </range>
+            </ray>
+        </sensor>
     </gazebo>
     <!-- ROS CONTROL -->
@@ -240,3 +280,8 @@
         </joint>
     </ros2_control>
+    <gazebo>
+        <plugin filename="gz_ros2_control-system" name="gz_ros2_control::GazeboSimROS2ControlPlugin">
+            <parameters>$(find chassis)/config/my_controllers.yaml</parameters>
+        </plugin>
+    </gazebo>
 </robot>

Commit message: added slam_toolbox config file

File: src/chassis/description/chassis_core.xacro (robot description, xacro)
@@ -20,4 +20,10 @@
     <!-- BASE LINK -->
     <link name="base_link"></link>
+    <joint name="base_footprint_joint" type="fixed">
+        <parent link="base_link"/>
+        <child link="base_footprint"/>
+        <origin xyz="0 0 0" rpy="0 0 0"/>
+    </joint>
+    <link name="base_footprint"></link>
     <!-- CHASSIS LINK -->
     <joint name="chassis_joint" type="fixed">

Commit message: changed coordinate handling

File: src/chassis/description/chassis_core.xacro (robot description, xacro)
@@ -19,11 +19,11 @@
     </material>
     <!-- BASE LINK -->
+    <link name="base_footprint"></link>
+    <joint name="base_link_joint" type="fixed">
+        <parent link="base_footprint"/>
+        <child link="base_link"/>
+        <origin xyz="0 0 0.075" rpy="0 0 0"/>
+    </joint>
     <link name="base_link"></link>
-    <joint name="base_footprint_joint" type="fixed">
-        <parent link="base_link"/>
-        <child link="base_footprint"/>
-        <origin xyz="0 0 0" rpy="0 0 0"/>
-    </joint>
-    <link name="base_footprint"></link>
     <!-- CHASSIS LINK -->
     <joint name="chassis_joint" type="fixed">

Commit message: added text logging to path planning

File: src/chassis/description/chassis_core.xacro (robot description, xacro)
@@ -19,11 +19,11 @@
     </material>
     <!-- BASE LINK -->
+    <link name="base_link"></link>
+    <joint name="base_footprint_joint" type="fixed">
+        <parent link="base_link"/>
+        <child link="base_footprint"/>
+        <origin xyz="0 0 0" rpy="0 0 0"/>
+    </joint>
     <link name="base_footprint"></link>
-    <joint name="base_link_joint" type="fixed">
-        <parent link="base_footprint"/>
-        <child link="base_link"/>
-        <origin xyz="0 0 0.075" rpy="0 0 0"/>
-    </joint>
-    <link name="base_link"></link>
     <!-- CHASSIS LINK -->
     <joint name="chassis_joint" type="fixed">
