Commit message: updated simulations

File: generated/cart_1.urdf (robot description, URDF)
Before this commit: robot simple_cart, 1 links, 0 joints
Links:
- link base_link: geometry collision box size=0.38 0.27 0.25; visual box size=0.38 0.27 0.25

File: generated/cart_2.urdf (robot description, URDF)
Before this commit: robot simple_cart, 1 links, 0 joints
Links:
- link base_link: geometry collision box size=0.38 0.27 0.25; visual box size=0.38 0.27 0.25

File: generated/cart_3.urdf (robot description, URDF)
Before this commit: robot simple_cart, 1 links, 0 joints
Links:
- link base_link: geometry collision box size=0.38 0.27 0.25; visual box size=0.38 0.27 0.25

File: src/intercart_comms/models/simple_cart/cart.urdf.xacro (robot description, xacro)
@@ -18,5 +18,5 @@
       <origin xyz="0 0 0.15"/>
       <geometry>
-        <box size="0.70 0.50 0.30"/>
+        <box size="0.38 0.27 0.25"/>
       </geometry>
       <material name="gray">
@@ -27,5 +27,5 @@
       <origin xyz="0 0 0.15"/>
       <geometry>
-        <box size="0.70 0.50 0.30"/>
+        <box size="0.38 0.27 0.25"/>
       </geometry>
     </collision>
